Commit message: [fix]修复了tf和参数映射的问题

File: src/rm_gimbal_description/urdf/rm_gimbal.urdf.xacro (robot description, xacro)
@@ -4,22 +4,23 @@
   <xacro:arg name="xyz" default="0.10 0 0.05" />
   <xacro:arg name="rpy" default="0 0 0" />
-  <link name="odom" />
+  <xacro:arg name="camera_name" default="camera" />
+  <link name="base_link" />
   <link name="gimbal_link" />
   <joint name="gimbal_joint" type="floating">
-    <parent link="odom" />
+    <parent link="base_link" />
     <child link="gimbal_link" />
   </joint>
-  <link name="camera_link" />
-  <joint name="camera_joint" type="fixed">
+  <link name="$(arg camera_name)_link" />
+  <joint name="$(arg camera_name)_joint" type="fixed">
     <origin xyz="$(arg xyz)" rpy="$(arg rpy)" />
     <parent link="gimbal_link" />
-    <child link="camera_link" />
+    <child link="$(arg camera_name)_link" />
     <axis xyz="0 0 0" />
   </joint>
-  <link name="camera_optical_frame" />
-  <joint name="camera_optical_joint" type="fixed">
+  <link name="$(arg camera_name)_optical_frame" />
+  <joint name="$(arg camera_name)_optical_joint" type="fixed">
     <origin xyz="0 0 0" rpy="${-pi/2} 0 ${-pi/2}" />
-    <parent link="camera_link" />
-    <child link="camera_optical_frame" />
+    <parent link="$(arg camera_name)_link" />
+    <child link="$(arg camera_name)_optical_frame" />
   </joint>
 </robot>

Commit message: [update]改了改tf的link名

File: src/rm_gimbal_description/urdf/rm_gimbal.urdf.xacro (robot description, xacro)
@@ -5,14 +5,14 @@
   <xacro:arg name="rpy" default="0 0 0" />
   <xacro:arg name="camera_name" default="camera" />
-  <link name="base_link" />
-  <link name="gimbal_link" />
-  <joint name="gimbal_joint" type="floating">
-    <parent link="base_link" />
-    <child link="gimbal_link" />
+  <link name="odom_omni" />
+  <link name="omni_gimbal_link" />
+  <joint name="omni_gimbal_joint" type="floating">
+    <parent link="odom_omni" />
+    <child link="omni_gimbal_link" />
   </joint>
   <link name="$(arg camera_name)_link" />
   <joint name="$(arg camera_name)_joint" type="fixed">
     <origin xyz="$(arg xyz)" rpy="$(arg rpy)" />
-    <parent link="gimbal_link" />
+    <parent link="omni_gimbal_link" />
     <child link="$(arg camera_name)_link" />
     <axis xyz="0 0 0" />
